File: pcb/beer2d2-pcb.sch (KiCad schematic (older format))
At the start: 5 parts

Commit message: ideas!
Parts:
- added C?: 0.1uF, ~, symbol C
- added C?: 1uF, ~, symbol C
- added IC?: TLC5971_SOP, ~, symbol TLC5971_SOP
- added LED? (x4): RGB-CA, ~, symbol LED_RGB-CA
- added LED? (x56): LED, ~, symbol LED
- added Q? (x8): NPN-BJT_SOT, ~, symbol NPN-BJT_SOT
- added R?: 2.2k, ~, symbol R
- added R? (x16): R, ~, symbol R
Connections:
- net COL0: now also LED?.2 (A), LED?.2 (A), LED?.2 (A), LED?.2 (A), LED?.2 (A), LED?.2 (A), LED?.2 (A), LED?.2 (A)
- net COL1: now also LED?.2 (A), LED?.2 (A), LED?.2 (A), LED?.2 (A), LED?.2 (A), LED?.2 (A), LED?.2 (A), LED?.2 (A)
- net COL2: now also LED?.2 (A), LED?.2 (A), LED?.2 (A), LED?.2 (A), LED?.2 (A), LED?.2 (A), LED?.2 (A), LED?.2 (A)
- net COL3: now also LED?.2 (A), LED?.2 (A), LED?.2 (A), LED?.2 (A), LED?.2 (A), LED?.2 (A), LED?.2 (A), LED?.2 (A)
- net COL4: now also LED?.2 (A), LED?.2 (A), LED?.2 (A), LED?.2 (A), LED?.2 (A), LED?.2 (A), LED?.2 (A), LED?.2 (A)
- net COL5: now also LED?.2 (A), LED?.2 (A), LED?.2 (A), LED?.2 (A), LED?.2 (A), LED?.2 (A), LED?.2 (A), LED?.2 (A)
- net COL6: now also LED?.2 (A), LED?.2 (A), LED?.2 (A), LED?.2 (A), LED?.2 (A), LED?.2 (A), LED?.2 (A), LED?.2 (A)
- net GND: now also C?.1, C?.2, IC?.0 (PAD), IC?.2 (GND), Q?.2 (E), Q?.2 (E), Q?.2 (E), Q?.2 (E), Q?.2 (E), Q?.2 (E), Q?.2 (E), Q?.2 (E), R?.1, R?.2, R?.2, R?.2, R?.2, R?.2, R?.2, R?.2, R?.2
- net ROW0: now also R?.1, R?.1, R?.1, R?.1, R?.1, R?.1, R?.1, R?.1
- net VCC: now also C?.1, C?.2, IC?.19 (VCC), IC?.20 (VREG), LED?.1 (A), LED?.1 (A), LED?.1 (A), LED?.1 (A)
- net BLU0 renamed TLC_SCK
- net TLC_SCK: now also IC?.10 (SCKI)
- net BLU1: no longer names the net of IC?.26 (PC3(ADC3/PCINT11))
- net GRN0 renamed TLC_SDA
- net TLC_SDA: now also IC?.9 (SDTI)
- net GRN1 renamed I2C_SDA
- net RED0: no longer names the net of IC?.25 (PC2(ADC2/PCINT10))
- net RED1 renamed I2C_SCL
- new net: IC?.1 (IREF), R?.2
- new net: IC?.13 (OUTR2), LED?.2 (R)
- new net: IC?.14 (OUTG2), LED?.3 (G)
- new net: IC?.15 (OUTB2), LED?.4 (B)
- new net: IC?.16 (OUTR3), LED?.2 (R)
- new net: IC?.17 (OUTG3), LED?.3 (G)
- new net: IC?.18 (OUTB3), LED?.4 (B)
- new net: IC?.3 (OUTR0), LED?.2 (R)
- new net: IC?.4 (OUTG0), LED?.3 (G)
- new net: IC?.5 (OUTB0), LED?.4 (B)
- new net: IC?.6 (OUTR1), LED?.2 (R)
- new net: IC?.7 (OUTG1), LED?.3 (G)
- new net: IC?.8 (OUTB1), LED?.4 (B)
- new net: Q?.1 (B), R?.1, R?.2 (x8)
- new net: LED?.1 (C), LED?.1 (C), LED?.1 (C), LED?.1 (C), LED?.1 (C), LED?.1 (C), LED?.1 (C), Q?.3 (C) (x8)
- no-connect marks 2 -> 7
Other:
- moved on the sheet: C?, IC?

Commit message: initial schematic pass
Parts:
- removed LED? (x4): RGB-CA, ~, symbol LED_RGB-CA
- removed LED? (x56): LED, ~, symbol LED
- removed Q? (x8): NPN-BJT_SOT, ~, symbol NPN-BJT_SOT
- removed R? (x16): R, ~, symbol R
- added C?: 10uF, ~, symbol C
- added C?: 1uF, ~, symbol C
- added IC?: VCC_REG, ~, symbol VCC_REG
- added J?: DCIN, ~, symbol DCIN
- added J?: PSI_BACK, ~, symbol 4PIN_FEMALE
- added J?: PSI_FRONT, ~, symbol 4PIN_FEMALE
- added J?: RGB_EXTRA, ~, symbol 4PIN_FEMALE
- added J?: EYE_FRONT, ~, symbol 4PIN_FEMALE
- added P?: AVR_ISP, ~, symbol AVR_ISP
- IC?: value ATMEGA328P_TQFP -> ATMEGA168P
Connections:
- net I2C_SCL is gone; now on net TLC_SCK: IC?.28 (PC5(ADC5/SCL/PCINT13))
- net I2C_SDA is gone; now on net TLC_SDA: IC?.27 (PC4(ADC4/SDA/PCINT12))
- net AVR_RST: now also P?.5 (RESET)
- net COL6: no longer IC?.7 (XTAL1(PB6))
- net GND: now also C?.1, C?.2, IC?.2 (COMMON), J?.2 (GND), P?.6 (GND)
- net TLC_SCK: no longer IC?.23 (PC0(ADC0/PCINT8))
- net TLC_SDA: no longer IC?.24 (PC1(ADC1/PCINT9))
- net VCC: now also IC?.3 (OUTPUT), P?.2 (VCC)
- net RED2: now reaches IC?.13 (OUTR2)
- net RED2: now also J?.1
- net GRN2: now reaches IC?.14 (OUTG2)
- net GRN2: now also J?.3
- net BLU2: now reaches IC?.15 (OUTB2)
- net BLU2: now also J?.4
- net RED3: now reaches IC?.16 (OUTR3)
- net RED3: now also J?.1
- net GRN3: now reaches IC?.17 (OUTG3)
- net GRN3: now also J?.3
- net BLU3: now reaches IC?.18 (OUTB3)
- net BLU3: now also J?.4
- net RED0: now reaches IC?.3 (OUTR0)
- net RED0: now also J?.1
- net GRN0: now reaches IC?.4 (OUTG0)
- net GRN0: now also J?.3
- net BLU0: now reaches IC?.5 (OUTB0)
- net BLU0: now also J?.4
- net RED1: now reaches IC?.6 (OUTR1)
- net RED1: now also J?.1
- net GRN1: now reaches IC?.7 (OUTG1)
- net GRN1: now also J?.3
- net BLU1: now reaches IC?.8 (OUTB1)
- net BLU1: now also J?.4
- net COL3 renamed AVR_MOSI
- net AVR_MOSI: now also P?.4 (MOSI)
- net COL4 renamed AVR_MISO
- net AVR_MISO: now also P?.1 (MISO)
- net COL5 renamed AVR_SCK
- net AVR_SCK: now also P?.3 (SCK)
- new net VIN: C?.2, IC?.1 (INPUT), J?.1 (VDC)
- new net VLED: J?.2, J?.2, J?.2, J?.2
- no-connect marks 7 -> 10
Other:
- note added: "RGB control (PSIs and eye)"
- note added: "front led panel"
- note added: "microcontroller"
- note added: "power"
- moved on the sheet: C?, IC?, R?
