File: pcb/beer2d2-front-pcb/beer2d2-front-pcb.kicad_pcb (KiCad board)
At the start: 2 copper layers, 81.9 x 50.8 mm, 178 parts, among them IC1 ATMEGA168P, IC2 VCC_REG, IC3 TLC5971_SOP, J1 PSI_FRONT, J2 EYE_FRONT, J3 PSI_BACK, J4 RGB_EXTRA, J5 DCIN, P1 AVR_ISP, Q1 MMBT4403, Q10 MMBT4401, Q11 MMBT4401, Q12 MMBT4403, Q13 MMBT4401, Q14 MMBT4403, Q15 MMBT4401, Q2 MMBT4403, Q3 MMBT4401, Q4 MMBT4401, Q5 MMBT4403, Q6 MMBT4403, Q7 MMBT4401, Q8 MMBT4401, Q9 MMBT4403

Commit message: taking another board pass
Routing:
- net VCC: track 199.4 -> 201.3 mm
Other:
- board size 81.9 x 50.8 mm -> 78.7 x 50.8 mm
Changed lines of the file:
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@@
   (general
     (links 302)
-    (no_connects 1)
+    (no_connects 0)
     (area 0 0 0 0)
     (thickness 1.6)
-    (drawings 16)
-    (tracks 1057)
+    (drawings 15)
+    (tracks 1058)
     (zones 0)
     (modules 178)
@@
     )
   )
-  (gr_line (start 132.715 238.76) (end 132.715 187.96) (angle 90) (layer Edge.Cuts) (width 0.1))
-  (gr_line (start 129.54 187.96) (end 129.54 238.76) (angle 90) (layer Edge.Cuts) (width 0.1))
-  (gr_line (start 211.455 187.96) (end 129.54 187.96) (angle 90) (layer Edge.Cuts) (width 0.1))
-  (gr_line (start 211.455 238.76) (end 211.455 187.96) (angle 90) (layer Edge.Cuts) (width 0.1))
-  (gr_line (start 129.54 238.76) (end 211.455 238.76) (angle 90) (layer Edge.Cuts) (width 0.1))
-  (dimension 75.565 (width 0.3) (layer Edge.Cuts)
-    (gr_text "2.9750 in" (at 167.3225 253.444999) (layer Edge.Cuts)
+  (dimension 50.8 (width 0.3) (layer Eco2.User)
+    (gr_text "2.0000 in" (at 126.92 213.36 90) (layer Eco2.User)
       (effects (font (size 1.5 1.5) (thickness 0.3)))
     )
-    (feature1 (pts (xy 205.105 247.65) (xy 205.105 254.794999)))
-    (feature2 (pts (xy 129.54 247.65) (xy 129.54 254.794999)))
-    (crossbar (pts (xy 129.54 252.094999) (xy 205.105 252.094999)))
-    (arrow1a (pts (xy 205.105 252.094999) (xy 203.978497 252.681419)))
-    (arrow1b (pts (xy 205.105 252.094999) (xy 203.978497 251.508579)))
-    (arrow2a (pts (xy 129.54 252.094999) (xy 130.666503 252.681419)))
-    (arrow2b (pts (xy 129.54 252.094999) (xy 130.666503 251.508579)))
+    (feature1 (pts (xy 130.81 187.96) (xy 125.57 187.96)))
+    (feature2 (pts (xy 130.81 238.76) (xy 125.57 238.76)))
+    (crossbar (pts (xy 128.27 238.76) (xy 128.27 187.96)))
+    (arrow1a (pts (xy 128.27 187.96) (xy 128.85642 189.086503)))
+    (arrow1b (pts (xy 128.27 187.96) (xy 127.68358 189.086503)))
+    (arrow2a (pts (xy 128.27 238.76) (xy 128.85642 237.633497)))
+    (arrow2b (pts (xy 128.27 238.76) (xy 127.68358 237.633497)))
   )
-  (dimension 63.5 (width 0.3) (layer Eco2.User)
-    (gr_text "2.5000 in" (at 161.29 246.459999) (layer Eco2.User)
+  (dimension 78.74 (width 0.3) (layer Eco2.User)
+    (gr_text "3.1000 in" (at 172.085 244.554999) (layer Eco2.User)
       (effects (font (size 1.5 1.5) (thickness 0.3)))
     )
-    (feature1 (pts (xy 193.04 240.03) (xy 193.04 247.809999)))
-    (feature2 (pts (xy 129.54 240.03) (xy 129.54 247.809999)))
-    (crossbar (pts (xy 129.54 245.109999) (xy 193.04 245.109999)))
-    (arrow1a (pts (xy 193.04 245.109999) (xy 191.913497 245.696419)))
-    (arrow1b (pts (xy 193.04 245.109999) (xy 191.913497 244.523579)))
-    (arrow2a (pts (xy 129.54 245.109999) (xy 130.666503 245.696419)))
-    (arrow2b (pts (xy 129.54 245.109999) (xy 130.666503 244.523579)))
+    (feature1 (pts (xy 211.455 240.665) (xy 211.455 245.904999)))
+    (feature2 (pts (xy 132.715 240.665) (xy 132.715 245.904999)))
+    (crossbar (pts (xy 132.715 243.204999) (xy 211.455 243.204999)))
+    (arrow1a (pts (xy 211.455 243.204999) (xy 210.328497 243.791419)))
+    (arrow1b (pts (xy 211.455 243.204999) (xy 210.328497 242.618579)))
+    (arrow2a (pts (xy 132.715 243.204999) (xy 133.841503 243.791419)))
+    (arrow2b (pts (xy 132.715 243.204999) (xy 133.841503 242.618579)))
   )
+  (gr_line (start 132.715 187.96) (end 211.455 187.96) (angle 90) (layer Edge.Cuts) (width 0.1))
+  (gr_line (start 132.715 238.76) (end 211.455 238.76) (angle 90) (layer Edge.Cuts) (width 0.1))
+  (gr_line (start 132.715 238.76) (end 132.715 187.96) (angle 90) (layer Edge.Cuts) (width 0.1))
+  (gr_line (start 211.455 238.76) (end 211.455 187.96) (angle 90) (layer Edge.Cuts) (width 0.1))
   (gr_line (start 178.435 187.96) (end 173.99 187.96) (angle 90) (layer Eco1.User) (width 0.2))
   (gr_line (start 178.435 210.185) (end 178.435 187.96) (angle 90) (layer Eco1.User) (width 0.2))
@@
   (segment (start 171.45 190.5) (end 171.45 192.47) (width 0.254) (layer F.Cu) (net 119))
   (segment (start 171.45 192.47) (end 170.88 193.04) (width 0.254) (layer F.Cu) (net 119))
+  (segment (start 198.69 191.135) (end 198.69 189.23) (width 0.254) (layer F.Cu) (net 120))
   (segment (start 200.66 192.532) (end 200.66 191.389) (width 0.254) (layer B.Cu) (net 120))
-  (segment (start 201.676 189.23) (end 197.485 189.23) (width 0.254) (layer B.Cu) (net 120))
-  (segment (start 201.93 189.484) (end 201.676 189.23) (width 0.254) (layer B.Cu) (net 120))
-  (segment (start 201.93 190.119) (end 201.93 189.484) (width 0.254) (layer B.Cu) (net 120))
+  (segment (start 200.66 192.532) (end 200.66 194.945) (width 0.254) (layer B.Cu) (net 120))
+  (segment (start 200.66 194.945) (end 201.93 196.215) (width 0.254) (layer B.Cu) (net 120))
+  (segment (start 201.93 196.215) (end 205.74 196.215) (width 0.254) (layer B.Cu) (net 120))
+  (segment (start 205.74 196.215) (end 206.375 195.58) (width 0.254) (layer B.Cu) (net 120))
+  (via (at 197.485 189.23) (size 0.762) (layers F.Cu B.Cu) (net 120))
+  (segment (start 198.69 189.23) (end 197.485 189.23) (width 0.254) (layer F.Cu) (net 120))
   (segment (start 200.66 191.389) (end 201.93 190.119) (width 0.254) (layer B.Cu) (net 120))
+  (segment (start 201.93 190.119) (end 201.93 189.484) (width 0.254) (layer B.Cu) (net 120))
+  (segment (start 201.93 189.484) (end 201.676 189.23) (width 0.254) (layer B.Cu) (net 120))
+  (segment (start 201.676 189.23) (end 197.485 189.23) (width 0.254) (layer B.Cu) (net 120))
   (segment (start 210.185 220.98) (end 210.185 221.234) (width 0.254) (layer F.Cu) (net 120))
   (segment (start 198.12 224.663) (end 198.12 225.425) (width 0.254) (layer F.Cu) (net 120))
@@
   (segment (start 201.865 207.01) (end 201.865 205.105) (width 0.254) (layer F.Cu) (net 120))
   (segment (start 201.865 208.091) (end 201.865 207.01) (width 0.254) (layer F.Cu) (net 120))
-  (segment (start 198.69 189.23) (end 197.485 189.23) (width 0.254) (layer F.Cu) (net 120))
-  (via (at 197.485 189.23) (size 0.762) (layers F.Cu B.Cu) (net 120))
-  (segment (start 205.74 196.215) (end 206.375 195.58) (width 0.254) (layer B.Cu) (net 120))
-  (segment (start 201.93 196.215) (end 205.74 196.215) (width 0.254) (layer B.Cu) (net 120))
-  (segment (start 200.66 194.945) (end 201.93 196.215) (width 0.254) (layer B.Cu) (net 120))
-  (segment (start 200.66 192.532) (end 200.66 194.945) (width 0.254) (layer B.Cu) (net 120))
   (segment (start 201.93 224.725) (end 201.93 220.345) (width 0.254) (layer F.Cu) (net 120))
   (segment (start 201.93 220.345) (end 201.295 219.71) (width 0.254) (layer F.Cu) (net 120))
@@
   (segment (start 189.295 203.9) (end 189.295 203.835) (width 0.254) (layer F.Cu) (net 120))
   (segment (start 196.475 190.75) (end 197.235 190.75) (width 0.254) (layer F.Cu) (net 120))
-  (segment (start 198.69 189.295) (end 198.69 189.23) (width 0.254) (layer F.Cu) (net 120))
   (segment (start 197.235 190.75) (end 198.69 189.295) (width 0.254) (layer F.Cu) (net 120))
+  (segment (start 198.69 189.295) (end 198.69 189.23) (width 0.254) (layer F.Cu) (net 120))
   (segment (start 196.475 191.4) (end 198.425 191.4) (width 0.254) (layer F.Cu) (net 120))
   (segment (start 198.425 191.4) (end 198.69 191.135) (width 0.254) (layer F.Cu) (net 120))
@@
   )
   (zone (net 16) (net_name /VIN) (layer F.Cu) (hatch edge 0.508)
-    (connect_pads (clearance 0.381))
+    (connect_pads yes (clearance 0.381))
     (min_thickness 0.381)
     (fill (arc_segments 16) (thermal_gap 0.508) (thermal_bridge_width 0.508))
@@
       (pts
         (xy 200.025 236.22) (xy 194.31 236.22) (xy 194.31 233.045) (xy 188.595 226.06) (xy 188.595 224.155)
-        (xy 194.31 224.155) (xy 194.31 226.695) (xy 200.025 233.68)
+        (xy 193.675 224.155) (xy 193.675 226.695) (xy 200.025 233.68)
       )
     )
   )
   (zone (net 120) (net_name VCC) (layer F.Cu) (hatch edge 0.508)
-    (connect_pads (clearance 0.381))
+    (connect_pads yes (clearance 0.381))
     (min_thickness 0.381)
     (fill (arc_segments 16) (thermal_gap 0.508) (thermal_bridge_width 0.508))
     (polygon
       (pts
-        (xy 202.565 225.425) (xy 201.295 225.425) (xy 199.39 226.06) (xy 197.485 226.06) (xy 196.85 223.52)
+        (xy 202.565 225.425) (xy 201.295 225.425) (xy 199.39 226.06) (xy 197.485 226.06) (xy 197.485 223.52)
         (xy 189.865 223.52) (xy 189.865 217.805) (xy 202.565 217.805)
       )
@@
   )
   (zone (net 47) (net_name GND) (layer F.Cu) (hatch edge 0.508)
-    (connect_pads (clearance 0.381))
-    (min_thickness 0.381)
+    (connect_pads (clearance 0.254))
+    (min_thickness 0.254)
     (fill (arc_segments 16) (thermal_gap 0.508) (thermal_bridge_width 0.508))
     (polygon
@@
       (pts        (xy 199.39 226.695) (xy 201.295 226.06) (xy 203.2 226.06) (xy 203.2 217.17) (xy 189.23 217.17)
         (xy 189.23 223.52) (xy 187.96 223.52) (xy 187.96 226.06) (xy 193.675 233.045) (xy 193.675 236.855)
-        (xy 200.66 236.855) (xy 200.66 233.045) (xy 194.945 226.695) (xy 194.945 224.155) (xy 196.215 224.155)
+        (xy 200.66 236.855) (xy 200.66 233.045) (xy 194.31 226.06) (xy 194.31 224.155) (xy 196.85 224.155)
         (xy 196.85 226.695)
       )

Commit message: liking this placement a lot more
Parts:
- removed C6: 0.1uF, 0603(1608m)
- removed the M3 at (135.9, 234.3)
- removed the M3 at (191.8, 234.3)
- removed the M3 at (135.9, 192.4)
- added M3: VAL**, M3, F.Cu at (249.6, 151.1)
- added M3: VAL**, M3, F.Cu at (189.2, 151.1)
- added M3: VAL**, M3, F.Cu at (189.9, 106.7)
- IC2: value VCC_REG -> 5VREG
- IC3: value TLC5971_SOP -> TLC5971
- Q1, Q12, Q14, Q2, Q5, Q6, Q9: value MMBT4403 -> 4403
- Q10, Q11, Q13, Q15, Q3, Q4, Q7, Q8: value MMBT4401 -> 4401
- moved J5 132.9 mm to (248.3, 110.0)
- moved C8 122.7 mm to (246.4, 116.8), turned to 0 degrees
- moved C7 118.8 mm to (250.2, 116.8), turned to 180 degrees
- moved IC2 116.7 mm to (248.3, 121.3)
- moved Q13 109.5 mm to (237.5, 116.8)
- moved R67 109.3 mm to (240.3, 116.8)
- moved R65 109.1 mm to (241.9, 116.8)
- moved Q10 107.8 mm to (237.5, 113.0)
- moved R54 107.6 mm to (240.3, 113.0)
- moved R43 107.5 mm to (241.9, 113.0)
- moved Q7 106.2 mm to (237.5, 109.2)
- moved R32 106.0 mm to (240.3, 109.2)
- moved R28 105.9 mm to (241.9, 109.2)
- moved Q3 104.6 mm to (237.5, 105.4)
- moved R16 104.4 mm to (240.3, 105.4)
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Routing:
- net (no net): track 0.00 -> 2220.3 mm, vias 0 -> 60
- net VCC: track 201.3 -> 0.00 mm, vias 10 -> 0
- net GND: track 113.6 -> 0.00 mm, vias 15 -> 0
- net /beer2d2 front LED panel/ROW4: track 72.7 -> 0.00 mm
- net /beer2d2 front LED panel/ROW3: track 72.7 -> 0.00 mm
- net /beer2d2 front LED panel/COL0: track 62.7 -> 0.00 mm
- net N-00000109: track 53.9 -> 0.00 mm, vias 2 -> 0
- net /beer2d2 front LED panel/ROW0: track 53.9 -> 0.00 mm
- net /beer2d2 front LED panel/ROW7: track 53.9 -> 0.00 mm
- net /beer2d2 front LED panel/ROW6: track 53.9 -> 0.00 mm
- net /beer2d2 front LED panel/ROW5: track 53.9 -> 0.00 mm
- net /beer2d2 front LED panel/ROW1: track 53.9 -> 0.00 mm
- net /beer2d2 front LED panel/ROW2: track 53.6 -> 0.00 mm
- net /RED0: track 53.0 -> 0.00 mm, vias 1 -> 0
- net N-00000104: track 51.3 -> 0.00 mm, vias 2 -> 0
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Other:
- board size 78.7 x 50.8 mm -> 120.7 x 135.3 mm

Commit message: about to redo a bunch of stuff
Parts:
- moved R31 1.52 mm to (239.6, 136.5)
- moved R14 1.27 mm to (241.3, 136.5)
- moved R30 1.02 mm to (243.0, 136.5)
- moved R45 0.76 mm to (244.6, 136.5)
- moved R66 0.51 mm to (246.3, 136.5)
- moved R78 0.25 mm to (247.9, 136.5)
- turned R44 to 270 degrees
Connections:
- M3 pad 1: (no net) -> GND (x3)
Routing:
- net (no net): track 2220.3 -> 0.00 mm, vias 60 -> 0
- net VCC: track 0.00 -> 187.4 mm, vias 0 -> 13
- net /beer2d2 front LED panel/ROW4: track 0.00 -> 76.9 mm
- net GND: track 0.00 -> 74.1 mm, vias 0 -> 16
- net /beer2d2 front LED panel/ROW3: track 0.00 -> 68.8 mm, vias 0 -> 2
- net /TLC_SDA: track 0.00 -> 66.5 mm, vias 0 -> 2
- net /TLC_SCK: track 0.00 -> 65.0 mm, vias 0 -> 2
- net N-00000109: track 0.00 -> 56.6 mm, vias 0 -> 2
- net /beer2d2 front LED panel/COL0: track 0.00 -> 56.3 mm
- net /beer2d2 front LED panel/ROW2: track 0.00 -> 53.7 mm
- net /beer2d2 front LED panel/ROW5: track 0.00 -> 53.7 mm
- net N-00000104: track 0.00 -> 52.2 mm, vias 0 -> 2
- net /beer2d2 front LED panel/ROW6: track 0.00 -> 52.1 mm
- net /beer2d2 front LED panel/ROW1: track 0.00 -> 52.0 mm
- net /beer2d2 front LED panel/ROW7: track 0.00 -> 50.4 mm
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Other:
- board size 120.7 x 135.3 mm -> 67.9 x 50.8 mm
