File: pcb/beer2d2-front-pcb/beer2d2-front-pcb_leds.sch (KiCad schematic (older format))
At the start: 157 parts

Commit message: first pass at board layout. will probably try again
Parts:
- removed Q?: MMBT4403, ~, symbol PNP-BJT_SOT
- added Q6: MMBT4403, ~, symbol PNP-BJT_SOT
- gave numbers to parts that had none: 156
Connections:
- net COL0: no longer R14.2
- net COL1: no longer R30.2
- net COL2: no longer R45.2
- net COL3: no longer R66.2
- net COL4: no longer R78.2
- net COL5: no longer R15.2
- net COL6: now also Q6.3 (C); no longer R31.2
- net ROW0: no longer R12.1
- net ROW1: no longer R28.1
- net ROW2: no longer R43.1
- net ROW3: no longer R65.1
- net ROW4: no longer R77.1
- net ROW5: no longer R13.1
- net ROW6: no longer R29.1
- net ROW7: no longer R44.1
- net VCC: now also Q6.2 (E)
- net at R27.2, R31.1: now also Q6.1 (B)
- new net AVR_C0: R14.2
- new net AVR_C1: R30.2
- new net AVR_C2: R45.2
- new net AVR_C3: R66.2
- new net AVR_C4: R78.2
- new net AVR_C5: R15.2
- new net AVR_C6: R31.2
- new net AVR_R0: R12.1
- new net AVR_R1: R28.1
- new net AVR_R2: R43.1
- new net AVR_R3: R65.1
- new net AVR_R4: R77.1
- new net AVR_R5: R13.1
- new net AVR_R6: R29.1
- new net AVR_R7: R44.1

Commit message: liking this placement a lot more
Parts:
- Q1, Q12, Q14, Q2, Q5, Q6, Q9: value MMBT4403 -> 4403
- Q10, Q11, Q13, Q15, Q3, Q4, Q7, Q8: value MMBT4401 -> 4401
Changed lines of the file:
@@
 P 1300 6600
 F 0 "Q1" H 1450 6750 60  0000 C CNN
-F 1 "MMBT4403" H 1100 6750 60  0000 C CNN
+F 1 "4403" H 1100 6750 60  0000 C CNN
 F 2 "~" H 1300 6600 60  0001 C CNN
 F 3 "~" H 1300 6600 60  0001 C CNN
@@
 U 1 1 52828A7E
 P 1900 4900
-F 0 "Q3" H 2000 5050 60  0000 C CNN
-F 1 "MMBT4401" H 1650 5050 60  0000 C CNN
+F 0 "Q3" H 1700 5100 60  0000 C CNN
+F 1 "4401" H 1750 5000 60  0000 C CNN
 F 2 "~" H 1900 4900 60  0001 C CNN
 F 3 "~" H 1900 4900 60  0001 C CNN
@@
 U 1 1 52828F59
 P 3750 4900
-F 0 "Q7" H 3850 5050 60  0000 C CNN
-F 1 "MMBT4401" H 3500 5050 60  0000 C CNN
+F 0 "Q7" H 3500 5100 60  0000 C CNN
+F 1 "4401" H 3550 5000 60  0000 C CNN
 F 2 "~" H 3750 4900 60  0001 C CNN
 F 3 "~" H 3750 4900 60  0001 C CNN
@@
 U 1 1 52828F86
 P 5600 4900
-F 0 "Q10" H 5700 5050 60  0000 C CNN
-F 1 "MMBT4401" H 5350 5050 60  0000 C CNN
+F 0 "Q10" H 5350 5100 60  0000 C CNN
+F 1 "4401" H 5400 5000 60  0000 C CNN
 F 2 "~" H 5600 4900 60  0001 C CNN
 F 3 "~" H 5600 4900 60  0001 C CNN
@@
 U 1 1 52828FB3
 P 7450 4900
-F 0 "Q13" H 7550 5050 60  0000 C CNN
-F 1 "MMBT4401" H 7200 5050 60  0000 C CNN
+F 0 "Q13" H 7250 5100 60  0000 C CNN
+F 1 "4401" H 7250 5000 60  0000 C CNN
 F 2 "~" H 7450 4900 60  0001 C CNN
 F 3 "~" H 7450 4900 60  0001 C CNN
@@
 U 1 1 52828FF0
 P 9300 4900
-F 0 "Q15" H 9400 5050 60  0000 C CNN
-F 1 "MMBT4401" H 9050 5050 60  0000 C CNN
+F 0 "Q15" H 9100 5100 60  0000 C CNN
+F 1 "4401" H 9100 5000 60  0000 C CNN
 F 2 "~" H 9300 4900 60  0001 C CNN
 F 3 "~" H 9300 4900 60  0001 C CNN
@@
 U 1 1 5282901D
 P 1900 5500
-F 0 "Q4" H 2000 5650 60  0000 C CNN
-F 1 "MMBT4401" H 1650 5650 60  0000 C CNN
+F 0 "Q4" H 1650 5700 60  0000 C CNN
+F 1 "4401" H 1700 5600 60  0000 C CNN
 F 2 "~" H 1900 5500 60  0001 C CNN
 F 3 "~" H 1900 5500 60  0001 C CNN
@@
 U 1 1 5282904A
 P 3750 5500
-F 0 "Q8" H 3850 5650 60  0000 C CNN
-F 1 "MMBT4401" H 3500 5650 60  0000 C CNN
+F 0 "Q8" H 3450 5700 60  0000 C CNN
+F 1 "4401" H 3500 5600 60  0000 C CNN
 F 2 "~" H 3750 5500 60  0001 C CNN
 F 3 "~" H 3750 5500 60  0001 C CNN
@@
 U 1 1 52829077
 P 5600 5500
-F 0 "Q11" H 5700 5650 60  0000 C CNN
-F 1 "MMBT4401" H 5350 5650 60  0000 C CNN
+F 0 "Q11" H 5350 5700 60  0000 C CNN
+F 1 "4401" H 5400 5600 60  0000 C CNN
 F 2 "~" H 5600 5500 60  0001 C CNN
 F 3 "~" H 5600 5500 60  0001 C CNN
@@
 P 3100 6600
 F 0 "Q5" H 3250 6750 60  0000 C CNN
-F 1 "MMBT4403" H 2900 6750 60  0000 C CNN
+F 1 "4403" H 2900 6750 60  0000 C CNN
 F 2 "~" H 3100 6600 60  0001 C CNN
 F 3 "~" H 3100 6600 60  0001 C CNN
@@
 P 4900 6600
 F 0 "Q9" H 5050 6750 60  0000 C CNN
-F 1 "MMBT4403" H 4700 6750 60  0000 C CNN
+F 1 "4403" H 4700 6750 60  0000 C CNN
 F 2 "~" H 4900 6600 60  0001 C CNN
 F 3 "~" H 4900 6600 60  0001 C CNN
@@
 P 6700 6600
 F 0 "Q12" H 6850 6750 60  0000 C CNN
-F 1 "MMBT4403" H 6500 6750 60  0000 C CNN
+F 1 "4403" H 6500 6750 60  0000 C CNN
 F 2 "~" H 6700 6600 60  0001 C CNN
 F 3 "~" H 6700 6600 60  0001 C CNN
@@
 P 8500 6600
 F 0 "Q14" H 8650 6750 60  0000 C CNN
-F 1 "MMBT4403" H 8300 6750 60  0000 C CNN
+F 1 "4403" H 8300 6750 60  0000 C CNN
 F 2 "~" H 8500 6600 60  0001 C CNN
 F 3 "~" H 8500 6600 60  0001 C CNN
@@
 P 1300 7300
 F 0 "Q2" H 1450 7450 60  0000 C CNN
-F 1 "MMBT4403" H 1100 7450 60  0000 C CNN
+F 1 "4403" H 1100 7450 60  0000 C CNN
 F 2 "~" H 1300 7300 60  0001 C CNN
 F 3 "~" H 1300 7300 60  0001 C CNN
@@
 P 3100 7300
 F 0 "Q6" H 3250 7450 60  0000 C CNN
-F 1 "MMBT4403" H 2900 7450 60  0000 C CNN
+F 1 "4403" H 2900 7450 60  0000 C CNN
 F 2 "~" H 3100 7300 60  0001 C CNN
 F 3 "~" H 3100 7300 60  0001 C CNN

Commit message: redoing front board
Parts:
- renumbered R2 to R1, R11 to R10, R12 to R11, R13 to R12, R14 to R13, R15 to R14, R16 to R15, R17 to R16, R18 to R17, R19 to R18, R20 to R19, R3 to R2, R21 to R20, R22 to R21, R23 to R22, R24 to R23, R25 to R24, R26 to R25, R27 to R26, R28 to R27, R29 to R28, R30 to R29, R4 to R3, R31 to R30, R32 to R31, R33 to R32, R34 to R33, R35 to R34, R36 to R35, R37 to R36, R38 to R37, R39 to R38, R40 to R39, R5 to R4, R41 to R40, R42 to R41, R43 to R42, R44 to R43, R45 to R44, R46 to R45, R47 to R46, R48 to R47, R49 to R48, R50 to R49, R6 to R5, R51 to R50, R52 to R51, R53 to R52, R54 to R53, R55 to R54, R56 to R55, R57 to R56, R58 to R57, R59 to R58, R60 to R59, R7 to R6, R61 to R60, R62 to R61, R63 to R62, R64 to R63, R65 to R64, R66 to R65, R67 to R66, R68 to R67, R69 to R68, R70 to R69, R8 to R7, R71 to R70, R72 to R71, R73 to R72, R74 to R73, R75 to R74, R76 to R75, R77 to R76, R78 to R77, R79 to R78, R80 to R79, R9 to R8, R81 to R80, R82 to R81, R83 to R82, R84 to R83, R85 to R84, R86 to R85, R87 to R86, R10 to R9

Commit message: layout complete
Parts:
- removed Q1, Q12, Q14, Q2, Q5, Q6, Q9: 4403, ~, symbol PNP-BJT_SOT
- removed Q10, Q11, Q13, Q15, Q3, Q4, Q7, Q8: 4401, ~, symbol NPN-BJT_SOT
- removed R10, R15, R16, R25, R26, R31, R32, R41, R53, R54, R55, R66, R75, R78, R9: 10kΩ, ~, symbol R
- removed R11, R12, R13, R14, R27, R28, R29, R30, R42, R43, R44, R64, R65, R76, R77: 1kΩ, ~, symbol R
- added Q1, Q10, Q13, Q2, Q5, Q6, Q9: DDTB113ZC, ~, symbol PNP-BJT-BIASED_SOT
- added Q11, Q12, Q14, Q15, Q3, Q4, Q7, Q8: DDTD113ZC, ~, symbol NPN-BJT-BIASED_SOT
Connections:
- net AVR_C0: now also Q1.1 (B)
- net AVR_C1: now also Q2.1 (B)
- net AVR_C2: now also Q5.1 (B)
- net AVR_C3: now also Q6.1 (B)
- net AVR_C4: now also Q9.1 (B)
- net AVR_C5: now also Q10.1 (B)
- net AVR_C6: now also Q13.1 (B)
- net AVR_R0: now also Q3.1 (B)
- net AVR_R1: now also Q4.1 (B)
- net AVR_R2: now also Q7.1 (B)
- net AVR_R3: now also Q8.1 (B)
- net AVR_R4: now also Q11.1 (B)
- net AVR_R5: now also Q12.1 (B)
- net AVR_R6: now also Q14.1 (B)
- net AVR_R7: now also Q15.1 (B)
- net COL0: now also Q1.3 (C)
- net COL1: now also Q2.3 (C)
- net COL2: now also Q5.3 (C)
- net COL3: now also Q6.3 (C)
- net COL4: now also Q9.3 (C)
- net COL5: now also Q10.3 (C)
- net COL6: now also Q13.3 (C)
- net GND: now also Q11.2 (E), Q12.2 (E), Q14.2 (E), Q15.2 (E), Q3.2 (E), Q4.2 (E), Q7.2 (E), Q8.2 (E)
- net ROW0: now also Q3.3 (C)
- net ROW1: now also Q4.3 (C)
- net ROW2: now also Q7.3 (C)
- net ROW3: now also Q8.3 (C)
- net ROW4: now also Q11.3 (C)
- net ROW5: now also Q12.3 (C)
- net ROW6: now also Q14.3 (C)
- net ROW7: now also Q15.3 (C)
- net VCC: now also Q1.2 (E), Q10.2 (E), Q13.2 (E), Q2.2 (E), Q5.2 (E), Q6.2 (E), Q9.2 (E)
