File: pcb/beer2d2-back-pcb/beer2d2-back-pcb.kicad_pcb (KiCad board)
At the start: 2 copper layers, 0 parts

Commit message: well, that wasn't so easy
Parts:
- added C1: 0.1uF, general sm:0603(1608m), F.Cu at (82.0, 144.8)
- added C10: 22pF, general sm:0603(1608m), F.Cu at (109.0, 125.7)
- added C11: 22pF, general sm:0603(1608m), F.Cu at (98.6, 134.0)
- added C12: 0.1uF, general sm:0603(1608m), F.Cu at (105.3, 133.0)
- added C13: 0.1uF, general sm:0603(1608m), F.Cu at (85.9, 152.0)
- added C14: 0.33uF, general sm:0603(1608m), F.Cu at (207.2, 54.5)
- added C15: 0.1uF, general sm:0603(1608m), F.Cu at (217.4, 52.9)
- added C2: 0.1uF, general sm:0603(1608m), F.Cu at (112.5, 133.0)
- added C3: 0.1uF, general sm:0603(1608m), F.Cu at (78.7, 152.0)
- added C4: 47pF, general sm:0603(1608m), F.Cu at (81.6, 159.3)
- added C5: 47pF, general sm:0603(1608m), F.Cu at (115.4, 125.7)
- added C6: 0.1uF, general sm:0603(1608m), F.Cu at (102.9, 141.2)
- added C7: 0.1uF, general sm:0603(1608m), F.Cu at (95.8, 148.5)
- added C8: 0.1uF, general sm:0603(1608m), F.Cu at (88.4, 159.3)
- added C9: 0.1uF, general sm:0603(1608m), F.Cu at (95.8, 141.2)
- added D1: 1N5819, sm leds:0603(1608m)_led, F.Cu at (83.3, 137.5)
- added F1: 500mA, general sm:1206(3216m), F.Cu at (94.2, 126.2)
- added IC1: 74HC238, small outline:TSSOP16, F.Cu at (85.3, 127.6)
- added IC2: TLC5971, small outline:HTSSOP20, F.Cu at (71.3, 150.4)
- added IC3: FT230X, small outline:SSOP16, F.Cu at (62.7, 149.3)
- added IC4: LM1117, small outline:SOT223, F.Cu at (219.6, 44.4)
- added IC5: ATMEGA328P, quad flat:TQFP32_7mm, F.Cu at (197.4, 47.6)
- added J1: USB, sm connectors:MICROUSB_sm, F.Cu at (46.3, 130.3)
- added J2: PSI1, single inline:SIP4, F.Cu at (59.8, 138.5)
- added J3: PSI2, single inline:SIP4, F.Cu at (71.9, 127.6)
- added J4: RGB1, single inline:SIP4, F.Cu at (58.4, 127.6)
- added J5: RGB2, single inline:SIP4, F.Cu at (50.4, 158.6)
- added J6: 6-12V, th connectors:2-PIN_SCREW-TERM_P200MIL, F.Cu at (208.4, 45.4)
- added LED1: RX, sm leds:0603(1608m)_led, F.Cu at (60.4, 159.3)
- added LED10: LED, th leds:LED-5mm, F.Cu at (68.9, 97.1)
- added LED11: LED, th leds:LED-5mm, F.Cu at (182.2, 125.1)
- added LED12: LED, th leds:LED-5mm, F.Cu at (74.6, 70.5)
- added LED13: LED, th leds:LED-5mm, F.Cu at (63.2, 79.4)
- added LED14: LED, th leds:LED-5mm, F.Cu at (57.5, 88.2)
- added LED15: LED, th leds:LED-5mm, F.Cu at (51.7, 61.6)
- added LED16: LED, th leds:LED-5mm, F.Cu at (57.5, 52.8)
- added LED17: LED, th leds:LED-5mm, F.Cu at (46.0, 70.5)
- added LED18: LED, th leds:LED-5mm, F.Cu at (51.7, 52.8)
- added LED19: LED, th leds:LED-5mm, F.Cu at (193.7, 125.1)
- added LED2: TX, sm leds:0603(1608m)_led, F.Cu at (69.8, 158.6)
- added LED20: LED, th leds:LED-5mm, F.Cu at (68.9, 79.4)
- added LED21: LED, th leds:LED-5mm, F.Cu at (91.7, 52.8)
- added LED22: LED, th leds:LED-5mm, F.Cu at (80.3, 61.6)
- added LED23: LED, th leds:LED-5mm, F.Cu at (57.5, 43.9)
- added LED24: LED, th leds:LED-5mm, F.Cu at (46.0, 61.6)
- added LED25: LED, th leds:LED-5mm, F.Cu at (51.7, 43.9)
- added LED26: LED, th leds:LED-5mm, F.Cu at (46.0, 52.8)
- added LED27: LED, th leds:LED-5mm, F.Cu at (97.4, 43.9)
- added LED28: LED, th leds:LED-5mm, F.Cu at (103.1, 43.9)
- added LED29: LED, th leds:LED-5mm, F.Cu at (86.0, 61.6)
- added LED3: LED, th leds:LED-5mm, F.Cu at (148.0, 125.1)
- added LED30: LED, th leds:LED-5mm, F.Cu at (91.7, 61.6)
- added LED31: LED, th leds:LED-5mm, F.Cu at (80.3, 70.5)
- added LED32: LED, th leds:LED-5mm, F.Cu at (63.2, 43.9)
- added LED33: LED, th leds:LED-5mm, F.Cu at (74.6, 52.8)
- added LED34: LED, th leds:LED-5mm, F.Cu at (63.2, 61.6)
- added LED35: LED, th leds:LED-5mm, F.Cu at (97.4, 52.8)
- added LED36: LED, th leds:LED-5mm, F.Cu at (103.1, 52.8)
- added LED37: LED, th leds:LED-5mm, F.Cu at (97.4, 61.6)
- added LED38: LED, th leds:LED-5mm, F.Cu at (68.9, 70.5)
- added LED39: LED, th leds:LED-5mm, F.Cu at (57.5, 70.5)
- added LED4: LED, th leds:LED-5mm, F.Cu at (148.0, 130.8)
- added LED40: LED, th leds:LED-5mm, F.Cu at (51.7, 79.4)
- added LED41: LED, th leds:LED-5mm, F.Cu at (68.9, 61.6)
- added LED42: LED, th leds:LED-5mm, F.Cu at (80.3, 43.9)
- added LED43: LED, th leds:LED-5mm, F.Cu at (86.0, 70.5)
- added LED44: LED, th leds:LED-5mm, F.Cu at (74.6, 79.4)
- added LED45: LED, th leds:LED-5mm, F.Cu at (80.3, 79.4)
- added LED46: LED, th leds:LED-5mm, F.Cu at (108.8, 43.9)
- added LED47: LED, th leds:LED-5mm, F.Cu at (86.0, 43.9)
- added LED48: LED, th leds:LED-5mm, F.Cu at (188.0, 125.1)
- added LED49: LED, th leds:LED-5mm, F.Cu at (91.7, 43.9)
- added LED5: LED, th leds:LED-5mm, F.Cu at (148.0, 136.5)
- added LED50: LED, th leds:LED-5mm, F.Cu at (80.3, 52.8)
- added LED51: LED, th leds:LED-5mm, F.Cu at (114.6, 43.9)
- added LED52: LED, th leds:LED-5mm, F.Cu at (63.2, 88.2)
- added LED53: LED, th leds:LED-5mm, F.Cu at (68.9, 88.2)
- added LED54: LED, th leds:LED-5mm, F.Cu at (57.5, 97.1)
- added LED55: LED, th leds:LED-5mm, F.Cu at (74.6, 61.6)
- added LED56: LED, th leds:LED-5mm, F.Cu at (63.2, 70.5)
- added LED57: LED, th leds:LED-5mm, F.Cu at (86.0, 52.8)
- added LED58: LED, th leds:LED-5mm, F.Cu at (57.5, 79.4)
- added LED59: LED, th leds:LED-5mm, F.Cu at (63.2, 97.1)
- added LED6: LED, th leds:LED-5mm, F.Cu at (148.0, 142.2)
- added LED60: LED, th leds:LED-5mm, F.Cu at (176.5, 125.1)
- added LED61: LED, th leds:LED-5mm, F.Cu at (228.0, 125.1)
- added LED62: LED, th leds:LED-5mm, F.Cu at (268.0, 125.1)
- added LED63: LED, th leds:LED-5mm, F.Cu at (51.7, 88.2)
- added LED64: LED, th leds:LED-5mm, F.Cu at (199.4, 125.1)
- added LED65: LED, th leds:LED-5mm, F.Cu at (210.8, 125.1)
- added LED66: LED, th leds:LED-5mm, F.Cu at (233.7, 125.1)
- added LED67: LED, th leds:LED-5mm, F.Cu at (250.8, 125.1)
- added LED68: LED, th leds:LED-5mm, F.Cu at (170.8, 125.1)
- added LED69: LED, th leds:LED-5mm, F.Cu at (74.6, 88.2)
- added LED7: LED, th leds:LED-5mm, F.Cu at (126.0, 43.9)
- added LED70: LED, th leds:LED-5mm, F.Cu at (46.0, 88.2)
- added LED71: LED, th leds:LED-5mm, F.Cu at (153.7, 125.1)
- added LED72: LED, th leds:LED-5mm, F.Cu at (262.3, 125.1)
- added LED73: LED, th leds:LED-5mm, F.Cu at (216.5, 125.1)
- added LED74: LED, th leds:LED-5mm, F.Cu at (256.5, 125.1)
- added LED75: LED, th leds:LED-5mm, F.Cu at (68.9, 52.8)
- added LED76: LED, th leds:LED-5mm, F.Cu at (51.7, 70.5)
- added LED77: LED, th leds:LED-5mm, F.Cu at (57.5, 61.6)
- added LED78: LED, th leds:LED-5mm, F.Cu at (63.2, 52.8)
- added LED79: LED, th leds:LED-5mm, F.Cu at (86.0, 79.4)
- added LED8: LED, th leds:LED-5mm, F.Cu at (165.1, 125.1)
- added LED80: LED, th leds:LED-5mm, F.Cu at (80.3, 88.2)
- added LED81: LED, th leds:LED-5mm, F.Cu at (222.2, 125.1)
- added LED82: LED, th leds:LED-5mm, F.Cu at (120.3, 43.9)
- added LED83: LED, th leds:LED-5mm, F.Cu at (74.6, 43.9)
- added LED84: LED, th leds:LED-5mm, F.Cu at (46.0, 79.4)
- added LED85: LED, th leds:LED-5mm, F.Cu at (68.9, 43.9)
- added LED86: LED, th leds:LED-5mm, F.Cu at (46.0, 43.9)
- added LED87: LED, th leds:LED-5mm, F.Cu at (74.6, 97.1)
- added LED88: LED, th leds:LED-5mm, F.Cu at (205.1, 125.1)
- added LED89: LED, th leds:LED-5mm, F.Cu at (239.4, 125.1)
- added LED9: LED, th leds:LED-5mm, F.Cu at (245.1, 125.1)
- added LED90: LED, th leds:LED-5mm, F.Cu at (159.4, 125.1)
- added P1: AVR_ISP, th connectors:2x3-array, F.Cu at (48.1, 146.0)
- added Q1: DDTD113ZC, small outline:SOT23, F.Cu at (170.3, 83.0)
- added Q10: DDTB113ZC, small outline:SOT23, F.Cu at (148.3, 98.9)
- added Q11: DDTB113ZC, small outline:SOT23, F.Cu at (154.4, 93.0)
- added Q12: DDTB113ZC, small outline:SOT23, F.Cu at (171.1, 71.3)
- added Q13: DDTB113ZC, small outline:SOT23, F.Cu at (164.2, 78.5)
- added Q14: DDTB113ZC, small outline:SOT23, F.Cu at (148.3, 93.0)
- added Q15: DDTB113ZC, small outline:SOT23, F.Cu at (107.5, 115.6)
- added Q16: DDTB113ZC, small outline:SOT23, F.Cu at (101.4, 115.6)
- added Q17: DDTB113ZC, small outline:SOT23, F.Cu at (130.0, 110.7)
- added Q18: DDTB113ZC, small outline:SOT23, F.Cu at (157.3, 85.8)
- added Q19: DDTB113ZC, small outline:SOT23, F.Cu at (177.2, 77.1)
- added Q2: DDTD113ZC, small outline:SOT23, F.Cu at (160.4, 91.6)
- added Q3: DDTD113ZC, small outline:SOT23, F.Cu at (148.2, 104.7)
- added Q4: DDTD113ZC, small outline:SOT23, F.Cu at (142.1, 109.1)
- added Q5: DDTD113ZC, small outline:SOT23, F.Cu at (154.4, 98.9)
- added Q6: DDTD113ZC, small outline:SOT23, F.Cu at (171.1, 77.1)
- added Q7: DDTD113ZC, small outline:SOT23, F.Cu at (177.2, 71.3)
- added Q8: DDTD113ZC, small outline:SOT23, F.Cu at (164.2, 84.4)
- added Q9: DDTB113ZC, small outline:SOT23, F.Cu at (136.0, 110.7)
- added R1: 2.2kΩ, general sm:0603(1608m), F.Cu at (102.1, 125.7)
- added R10: 110Ω, general sm:0603(1608m), F.Cu at (120.9, 60.8)
- added R11: 110Ω, general sm:0603(1608m), F.Cu at (123.2, 82.5)
- added R12: 110Ω, general sm:0603(1608m), F.Cu at (153.0, 50.3)
- added R13: 110Ω, general sm:0603(1608m), F.Cu at (116.3, 76.9)
- added R14: 110Ω, general sm:0603(1608m), F.Cu at (146.1, 50.3)
- added R15: 110Ω, general sm:0603(1608m), F.Cu at (53.5, 114.0)
- added R16: 110Ω, general sm:0603(1608m), F.Cu at (122.1, 68.0)
- added R17: 110Ω, general sm:0603(1608m), F.Cu at (139.2, 50.3)
- added R18: 110Ω, general sm:0603(1608m), F.Cu at (144.9, 43.0)
- added R19: 110Ω, general sm:0603(1608m), F.Cu at (176.1, 57.5)
- added R2: 10kΩ, general sm:0603(1608m), F.Cu at (88.9, 144.8)
- added R20: 110Ω, general sm:0603(1608m), F.Cu at (130.4, 104.3)
- added R21: 110Ω, general sm:0603(1608m), F.Cu at (170.4, 64.8)
- added R22: 110Ω, general sm:0603(1608m), F.Cu at (141.8, 95.4)
- added R23: 110Ω, general sm:0603(1608m), F.Cu at (115.2, 69.7)
- added R24: 110Ω, general sm:0603(1608m), F.Cu at (98.0, 87.4)
- added R25: 110Ω, general sm:0603(1608m), F.Cu at (138.0, 43.0)
- added R26: 110Ω, general sm:0603(1608m), F.Cu at (123.2, 75.3)
- added R27: 110Ω, general sm:0603(1608m), F.Cu at (164.6, 72.0)
- added R28: 110Ω, general sm:0603(1608m), F.Cu at (177.3, 64.8)
- added R29: 110Ω, general sm:0603(1608m), F.Cu at (137.3, 102.7)
- added R3: 27Ω, general sm:0603(1608m), F.Cu at (75.7, 159.3)
- added R30: 110Ω, general sm:0603(1608m), F.Cu at (142.8, 64.8)
- added R31: 110Ω, general sm:0603(1608m), F.Cu at (148.5, 57.5)
- added R32: 110Ω, general sm:0603(1608m), F.Cu at (94.9, 110.8)
- added R33: 110Ω, general sm:0603(1608m), F.Cu at (111.8, 85.8)
- added R34: 110Ω, general sm:0603(1608m), F.Cu at (95.9, 103.5)
- added R35: 110Ω, general sm:0603(1608m), F.Cu at (172.5, 43.0)
- added R36: 110Ω, general sm:0603(1608m), F.Cu at (114.2, 93.0)
- added R37: 110Ω, general sm:0603(1608m), F.Cu at (109.7, 101.9)
- added R38: 110Ω, general sm:0603(1608m), F.Cu at (102.8, 109.1)
- added R39: 110Ω, general sm:0603(1608m), F.Cu at (134.7, 59.2)
- added R4: 27Ω, general sm:0603(1608m), F.Cu at (92.6, 134.0)
- added R40: 110Ω, general sm:0603(1608m), F.Cu at (89.0, 103.5)
- added R41: 110Ω, general sm:0603(1608m), F.Cu at (81.1, 112.4)
- added R42: 110Ω, general sm:0603(1608m), F.Cu at (151.8, 43.0)
- added R43: 110Ω, general sm:0603(1608m), F.Cu at (137.0, 73.7)
- added R44: 110Ω, general sm:0603(1608m), F.Cu at (155.4, 57.5)
- added R45: 110Ω, general sm:0603(1608m), F.Cu at (102.8, 101.9)
- added R46: 110Ω, general sm:0603(1608m), F.Cu at (109.7, 109.1)
- added R47: 110Ω, general sm:0603(1608m), F.Cu at (129.0, 68.0)
- added R48: 110Ω, general sm:0603(1608m), F.Cu at (100.4, 94.6)
- added R49: 110Ω, general sm:0603(1608m), F.Cu at (88.0, 112.4)
- added R5: 1kΩ, general sm:0603(1608m), F.Cu at (102.0, 148.5)
- added R50: 110Ω, general sm:0603(1608m), F.Cu at (141.6, 57.5)
- added R51: 110Ω, general sm:0603(1608m), F.Cu at (143.9, 72.0)
- added R52: 110Ω, general sm:0603(1608m), F.Cu at (137.0, 80.9)
- added R53: 110Ω, general sm:0603(1608m), F.Cu at (179.4, 43.0)
- added R54: 110Ω, general sm:0603(1608m), F.Cu at (143.9, 79.3)
- added R55: 110Ω, general sm:0603(1608m), F.Cu at (158.7, 43.0)
- added R56: 110Ω, general sm:0603(1608m), F.Cu at (135.9, 66.4)
- added R57: 110Ω, general sm:0603(1608m), F.Cu at (130.1, 75.3)
- added R58: 110Ω, general sm:0603(1608m), F.Cu at (127.8, 60.8)
- added R59: 110Ω, general sm:0603(1608m), F.Cu at (162.3, 57.5)
- added R6: 1kΩ, general sm:0603(1608m), F.Cu at (109.1, 140.2)
- added R60: 110Ω, general sm:0603(1608m), F.Cu at (121.1, 97.0)
- added R61: 110Ω, general sm:0603(1608m), F.Cu at (121.1, 89.8)
- added R62: 110Ω, general sm:0603(1608m), F.Cu at (107.3, 94.6)
- added R63: 110Ω, general sm:0603(1608m), F.Cu at (75.2, 105.1)
- added R64: 110Ω, general sm:0603(1608m), F.Cu at (67.3, 114.0)
- added R65: 110Ω, general sm:0603(1608m), F.Cu at (132.3, 51.9)
- added R66: 110Ω, general sm:0603(1608m), F.Cu at (46.6, 114.0)
- added R67: 110Ω, general sm:0603(1608m), F.Cu at (165.6, 43.0)
- added R68: 110Ω, general sm:0603(1608m), F.Cu at (166.8, 50.3)
- added R69: 110Ω, general sm:0603(1608m), F.Cu at (150.8, 72.0)
- added R7: 110Ω, general sm:0603(1608m), F.Cu at (74.2, 114.0)
- added R70: 110Ω, general sm:0603(1608m), F.Cu at (156.6, 64.8)
- added R71: 110Ω, general sm:0603(1608m), F.Cu at (82.1, 105.1)
- added R72: 110Ω, general sm:0603(1608m), F.Cu at (93.5, 96.3)
- added R73: 110Ω, general sm:0603(1608m), F.Cu at (104.9, 87.4)
- added R74: 110Ω, general sm:0603(1608m), F.Cu at (60.4, 114.0)
- added R75: 110Ω, general sm:0603(1608m), F.Cu at (128.0, 89.8)
- added R76: 110Ω, general sm:0603(1608m), F.Cu at (149.7, 64.8)
- added R77: 110Ω, general sm:0603(1608m), F.Cu at (130.1, 82.5)
- added R78: 110Ω, general sm:0603(1608m), F.Cu at (159.9, 50.3)
- added R79: 110Ω, general sm:0603(1608m), F.Cu at (173.7, 50.3)
- added R8: 110Ω, general sm:0603(1608m), F.Cu at (109.4, 78.5)
- added R80: 110Ω, general sm:0603(1608m), F.Cu at (128.0, 97.0)
- added R81: 110Ω, general sm:0603(1608m), F.Cu at (116.6, 104.3)
- added R82: 110Ω, general sm:0603(1608m), F.Cu at (123.5, 104.3)
- added R83: 110Ω, general sm:0603(1608m), F.Cu at (134.9, 95.4)
- added R84: 110Ω, general sm:0603(1608m), F.Cu at (157.7, 79.3)
- added R85: 110Ω, general sm:0603(1608m), F.Cu at (150.8, 86.5)
- added R86: 110Ω, general sm:0603(1608m), F.Cu at (123.5, 111.5)
- added R87: 110Ω, general sm:0603(1608m), F.Cu at (116.6, 111.5)
- added R88: 110Ω, general sm:0603(1608m), F.Cu at (150.8, 79.3)
- added R89: 110Ω, general sm:0603(1608m), F.Cu at (157.7, 72.0)
- added R9: 110Ω, general sm:0603(1608m), F.Cu at (86.6, 96.3)
- added R90: 110Ω, general sm:0603(1608m), F.Cu at (180.6, 50.3)
- added R91: 110Ω, general sm:0603(1608m), F.Cu at (143.9, 86.5)
- added R92: 110Ω, general sm:0603(1608m), F.Cu at (163.5, 64.8)
- added R93: 110Ω, general sm:0603(1608m), F.Cu at (169.2, 57.5)
- added R94: 110Ω, general sm:0603(1608m), F.Cu at (137.0, 88.2)
- added Y1: 16MHz, crystals:HC49, F.Cu at (72.5, 138.7)
Other:
- net class Default: via_dia 0.889 -> 0.762; via_drill 0.635 -> 0.381
- rule trace_min: 0.254 -> 0.1524
- rule via_min_drill: 0.508 -> 0.3302
- rule via_min_size: 0.889 -> 0.6858
